File: Schematic/Schematic.kicad_pcb (KiCad board)
At the start: 2 copper layers, 13 parts, among them IC1 ATMEGA328-P, P1 Arduino Programmer, P2 X8R, P3 Motors, P4 Motors Voltage, U1 LM7805, U3 SN754410, Y1 Resonator

Commit message: Rx power pins
Parts:
- added P5: Rx PS, Connectors_Molex:Molex_KK-6410-02_02x2.54mm_Straight, F.Cu at (224.2, 128.9)
- moved P2 4.44 mm to (224.2, 141.0)
Routing:
- net +5V: track 101.8 -> 107.0 mm
Changed lines of the file:
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@@
 (kicad_pcb (version 4) (host pcbnew 4.0.4-stable)
   (general
-    (links 42)
+    (links 44)
     (no_connects 0)
-    (area 164.364999 86.894999 230.605001 146.785001)
+    (area 164.364999 75.17 230.605001 146.785001)
     (thickness 1.6)
     (drawings 5)
-    (tracks 128)
+    (tracks 130)
     (zones 0)
-    (modules 13)
+    (modules 14)
     (nets 31)
   )
   (page A4)
   (layers
-    (0 F.Cu signal)
+    (0 F.Cu signal hide)
     (31 B.Cu signal)
     (32 B.Adhes user hide)
@@
   )
   (module Connectors_Molex:Molex_KK-6410-03_03x2.54mm_Straight (layer F.Cu)
-    (at 224.155 136.525 90)
+    (at 224.155 140.97 90)
     (descr "Connector Headers with Friction Lock, 22-27-2031, http://www.molex.com/pdm_docs/sd/022272021_sd.pdf")
     (tags "connector molex kk_6410 22-27-2031")
@@
     )
   )
+  (module Connectors_Molex:Molex_KK-6410-02_02x2.54mm_Straight (layer F.Cu)
+    (at 224.155 128.905 270)
+    (descr "Connector Headers with Friction Lock, 22-27-2021, http://www.molex.com/pdm_docs/sd/022272021_sd.pdf")
+    (tags "connector molex kk_6410 22-27-2021")
+    (fp_text reference P5 (at 1 -4.5 270) (layer F.SilkS)
+      (effects (font (size 1 1) (thickness 0.15)))
+    )
+    (fp_text value "Rx PS" (at 1.27 4.5 270) (layer F.Fab)
+      (effects (font (size 1 1) (thickness 0.15)))
+    )
+    (fp_line (start -1.37 -3.02) (end -1.37 2.98) (layer F.SilkS) (width 0.12))
+    (fp_line (start -1.37 2.98) (end 3.91 2.98) (layer F.SilkS) (width 0.12))
+    (fp_line (start 3.91 2.98) (end 3.91 -3.02) (layer F.SilkS) (width 0.12))
+    (fp_line (start 3.91 -3.02) (end -1.37 -3.02) (layer F.SilkS) (width 0.12))
+    (fp_line (start 0 2.98) (end 0 1.98) (layer F.SilkS) (width 0.12))
+    (fp_line (start 0 1.98) (end 2.54 1.98) (layer F.SilkS) (width 0.12))
+    (fp_line (start 2.54 1.98) (end 2.54 2.98) (layer F.SilkS) (width 0.12))
+    (fp_line (start 0 1.98) (end 0.25 1.55) (layer F.SilkS) (width 0.12))
+    (fp_line (start 0.25 1.55) (end 2.29 1.55) (layer F.SilkS) (width 0.12))
+    (fp_line (start 2.29 1.55) (end 2.54 1.98) (layer F.SilkS) (width 0.12))
+    (fp_line (start 0.25 2.98) (end 0.25 1.98) (layer F.SilkS) (width 0.12))
+    (fp_line (start 2.29 2.98) (end 2.29 1.98) (layer F.SilkS) (width 0.12))
+    (fp_line (start -0.8 -3.02) (end -0.8 -2.4) (layer F.SilkS) (width 0.12))
+    (fp_line (start -0.8 -2.4) (end 0.8 -2.4) (layer F.SilkS) (width 0.12))
+    (fp_line (start 0.8 -2.4) (end 0.8 -3.02) (layer F.SilkS) (width 0.12))
+    (fp_line (start 1.74 -3.02) (end 1.74 -2.4) (layer F.SilkS) (width 0.12))
+    (fp_line (start 1.74 -2.4) (end 3.34 -2.4) (layer F.SilkS) (width 0.12))
+    (fp_line (start 3.34 -2.4) (end 3.34 -3.02) (layer F.SilkS) (width 0.12))
+    (fp_line (start -1.9 3.5) (end -1.9 -3.55) (layer F.CrtYd) (width 0.05))
+    (fp_line (start -1.9 -3.55) (end 4.45 -3.55) (layer F.CrtYd) (width 0.05))
+    (fp_line (start 4.45 -3.55) (end 4.45 3.5) (layer F.CrtYd) (width 0.05))
+    (fp_line (start 4.45 3.5) (end -1.9 3.5) (layer F.CrtYd) (width 0.05))
+    (pad 1 thru_hole rect (at 0 0 270) (size 2 2.6) (drill 1.2) (layers *.Cu *.Mask)
+      (net 3 +5V))
+    (pad 2 thru_hole oval (at 2.54 0 270) (size 2 2.6) (drill 1.2) (layers *.Cu *.Mask)
+      (net 2 GND))
+  )
   (gr_line (start 164.465 146.685) (end 164.465 143.51) (angle 90) (layer Eco1.User) (width 0.2))
   (gr_line (start 230.505 146.685) (end 164.465 146.685) (angle 90) (layer Eco1.User) (width 0.2))
@@
   (segment (start 184.15 95.885) (end 191.77 95.885) (width 0.35) (layer B.Cu) (net 1))
   (segment (start 208.915 123.19) (end 209.55 123.19) (width 0.35) (layer B.Cu) (net 2))
+  (segment (start 224.155 128.905) (end 224.155 126.365) (width 0.35) (layer B.Cu) (net 3) (status 400000))
+  (segment (start 224.155 126.365) (end 222.25 124.46) (width 0.35) (layer B.Cu) (net 3) (status 800000))
   (segment (start 191.77 113.03) (end 194.945 113.03) (width 0.35) (layer B.Cu) (net 3))
   (segment (start 196.85 99.695) (end 196.85 95.885) (width 0.35) (layer B.Cu) (net 3))
@@
   (segment (start 213.36 105.41) (end 215.265 103.505) (width 0.35) (layer B.Cu) (net 4))
   (segment (start 201.295 105.41) (end 209.55 105.41) (width 0.35) (layer B.Cu) (net 4))
-  (segment (start 217.17 138.43) (end 218.44 138.43) (width 0.35) (layer B.Cu) (net 5))
-  (segment (start 220.345 136.525) (end 224.155 136.525) (width 0.35) (layer B.Cu) (net 5))
-  (segment (start 218.44 138.43) (end 220.345 136.525) (width 0.35) (layer B.Cu) (net 5))
+  (segment (start 217.17 138.43) (end 218.44 138.43) (width 0.35) (layer B.Cu) (net 5) (status 400000))
+  (segment (start 220.98 140.97) (end 224.155 140.97) (width 0.35) (layer B.Cu) (net 5) (status 800000))
+  (segment (start 218.44 138.43) (end 220.98 140.97) (width 0.35) (layer B.Cu) (net 5))
   (segment (start 201.295 107.95) (end 209.55 107.95) (width 0.35) (layer B.Cu) (net 6))
-  (segment (start 217.17 135.89) (end 218.44 135.89) (width 0.35) (layer B.Cu) (net 7))
-  (segment (start 220.345 133.985) (end 224.155 133.985) (width 0.35) (layer B.Cu) (net 7))
-  (segment (start 218.44 135.89) (end 220.345 133.985) (width 0.35) (layer B.Cu) (net 7))
+  (segment (start 217.17 135.89) (end 218.44 135.89) (width 0.35) (layer B.Cu) (net 7) (status 400000))
+  (segment (start 220.98 138.43) (end 224.155 138.43) (width 0.35) (layer B.Cu) (net 7) (status 800000))
+  (segment (start 218.44 135.89) (end 220.98 138.43) (width 0.35) (layer B.Cu) (net 7))
   (segment (start 201.295 110.49) (end 209.55 110.49) (width 0.35) (layer B.Cu) (net 8))
-  (segment (start 217.17 133.35) (end 218.44 133.35) (width 0.35) (layer B.Cu) (net 9))
-  (segment (start 220.345 131.445) (end 224.155 131.445) (width 0.35) (layer B.Cu) (net 9))
-  (segment (start 218.44 133.35) (end 220.345 131.445) (width 0.35) (layer B.Cu) (net 9))
+  (segment (start 217.17 133.35) (end 218.44 133.35) (width 0.35) (layer B.Cu) (net 9) (status 400000))
+  (segment (start 220.98 135.89) (end 224.155 135.89) (width 0.35) (layer B.Cu) (net 9) (status 800000))
+  (segment (start 218.44 133.35) (end 220.98 135.89) (width 0.35) (layer B.Cu) (net 9))
   (segment (start 191.77 128.27) (end 196.85 128.27) (width 0.35) (layer B.Cu) (net 10))
   (segment (start 200.66 113.03) (end 209.55 113.03) (width 0.35) (layer B.Cu) (net 10))
@@
   (segment (start 206.375 128.27) (end 209.55 128.27) (width 0.35) (layer B.Cu) (net 17))
   (segment (start 205.105 127) (end 206.375 128.27) (width 0.35) (layer B.Cu) (net 17))
-  (segment (start 184.15 113.03) (end 173.355 113.03) (width 0.35) (layer B.Cu) (net 19) (status 400000))
-  (segment (start 203.2 130.81) (end 209.55 130.81) (width 0.35) (layer B.Cu) (net 19) (status 800000))
+  (segment (start 184.15 113.03) (end 173.355 113.03) (width 0.35) (layer B.Cu) (net 19))
+  (segment (start 203.2 130.81) (end 209.55 130.81) (width 0.35) (layer B.Cu) (net 19))
   (segment (start 203.2 133.35) (end 203.2 130.81) (width 0.35) (layer B.Cu) (net 19))
   (via (at 203.2 133.35) (size 0.6) (drill 0.4) (layers F.Cu B.Cu) (net 19))
@@
   (segment (start 168.91 117.475) (end 168.91 137.16) (width 0.35) (layer B.Cu) (net 19))
   (segment (start 173.355 113.03) (end 168.91 117.475) (width 0.35) (layer B.Cu) (net 19))
-  (segment (start 184.15 115.57) (end 173.355 115.57) (width 0.35) (layer B.Cu) (net 21) (status 400000))
-  (segment (start 205.74 133.35) (end 209.55 133.35) (width 0.35) (layer B.Cu) (net 21) (status 800000))
+  (segment (start 184.15 115.57) (end 173.355 115.57) (width 0.35) (layer B.Cu) (net 21))
+  (segment (start 205.74 133.35) (end 209.55 133.35) (width 0.35) (layer B.Cu) (net 21))
   (via (at 205.74 133.35) (size 0.6) (drill 0.4) (layers F.Cu B.Cu) (net 21))
   (segment (start 205.74 139.065) (end 205.74 133.35) (width 0.35) (layer F.Cu) (net 21))
@@
   (segment (start 180.975 125.73) (end 184.15 125.73) (width 0.35) (layer B.Cu) (net 28))
   (segment (start 179.07 123.825) (end 180.975 125.73) (width 0.35) (layer B.Cu) (net 28))
-  (segment (start 191.77 118.11) (end 193.675 118.11) (width 0.35) (layer B.Cu) (net 29) (status 400000))
-  (segment (start 173.99 126.365) (end 175.895 126.365) (width 0.35) (layer B.Cu) (net 29) (status 800000))
+  (segment (start 191.77 118.11) (end 193.675 118.11) (width 0.35) (layer B.Cu) (net 29))
+  (segment (start 173.99 126.365) (end 175.895 126.365) (width 0.35) (layer B.Cu) (net 29))
   (segment (start 172.72 127.635) (end 173.99 126.365) (width 0.35) (layer B.Cu) (net 29))
   (segment (start 172.72 135.255) (end 172.72 127.635) (width 0.35) (layer B.Cu) (net 29))
